File: pypilot_controller.kicad_pcb (KiCad board)
At the start: 2 copper layers, 90 x 54 mm, 22 parts, among them J2 12V, J3 GND, J4 OUTA, J5 OUTB, J6 CAN-HI, J7 CAN-LO, P1 Digital, P2 Analog, P3 CONN_01X01, P4 CONN_01X01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

Commit message: many changes
Parts:
- added D1: PMEG3020EH, Diodes_SMD:D_SOD-123F, F.Cu at (190.3, 103.5)
- added F1: 15A, CustomComponents:atm_fuse_holder-mpd-bk-6013, F.Cu at (191.8, 110.8)
- added H6: MountingHole, Mounting_Holes:MountingHole_3.2mm_M3, F.Cu at (113.9, 63.8)
- added H7: MountingHole, Mounting_Holes:MountingHole_3.2mm_M3, F.Cu at (114.0, 110.0)
- added H8: MountingHole, Mounting_Holes:MountingHole_3.2mm_M3, F.Cu at (195.0, 64.0)
- added H9: MountingHole, Mounting_Holes:MountingHole_3.2mm_M3, F.Cu at (165.0, 110.0)
- added J1: Right Rudder Stop, Connectors_JST:JST_XH_B02B-XH-A_02x2.50mm_Straight, F.Cu at (113.5, 75.5)
- added J8: Left Rudder Stop, Connectors_JST:JST_XH_B02B-XH-A_02x2.50mm_Straight, F.Cu at (113.5, 99.7)
- moved J7 78.3 mm to (122.3, 106.1), turned to 0 degrees
- moved J6 75.4 mm to (130.2, 106.1), turned to 0 degrees
- moved J4 21.4 mm to (194.0, 89.3)
- moved J5 19.5 mm to (194.0, 82.2)
- moved J3 8.70 mm to (194.0, 75.1)
- moved J2 4.40 mm to (193.9, 97.0)
- moved U3 1.96 mm to (172.3, 87.4)
Connections:
- J2 pad 1: +12V -> Net-(F1-Pad1)
- P1 pad 10: (no net) -> D7
- P1 pad 11: (no net) -> D8
- P2 pad 1: (no net) -> /Vin
Routing:
- net CANH: track 121.3 -> 16.5 mm, vias 1 -> 0
- net CANL: track 115.1 -> 12.2 mm, vias 1 -> 0
- net D7: track 0.00 -> 84.7 mm, vias 0 -> 1
- net /Vin: track 0.00 -> 61.0 mm
- net D8: track 0.00 -> 51.1 mm, vias 0 -> 1
- net A1: track 0.00 -> 35.9 mm
- net Net-(F1-Pad1): track 0.00 -> 23.1 mm
- net Reset: track 20.4 -> 35.6 mm, vias 1 -> 2
- net OUTB: track 30.0 -> 44.4 mm
- net OUTA: track 24.4 -> 35.3 mm
- net D3: track 38.5 -> 45.9 mm
- net D4: track 49.8 -> 56.7 mm, vias 0 -> 1
- net D6: track 51.5 -> 56.5 mm, vias 1 -> 0
- net D5: track 46.2 -> 42.2 mm, vias 1 -> 0
- net +5V: track 89.7 -> 86.3 mm, vias 0 -> 2
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Other:
- board text added: "Left Rudder"
- board text added: "Rev A"
- board text added: "Right Rudder"
- board text added: "http://bit-builder.com pypilot controller"

Commit message: Crystal was wired incorrectly
Replaced schematic symbol
Fixed pcb layout
incremented revision to B
Connections:
- Y1 pad 2: Net-(C4-Pad1) -> GND
- Y1 pad 3: (no net) -> Net-(C4-Pad1)
- Y1 pad 4: (no net) -> GND
Routing:
- net Net-(C4-Pad1): track 11.6 -> 10.3 mm
- net Net-(C3-Pad1): track 9.32 -> 9.98 mm
Other:
- board text added: "Rev B"
- board text removed: "Rev A"
