File: pypilot_controller.sch (KiCad schematic (older format))
At the start: 22 parts, among them J2 12V, J3 GND, J4 OUTA, J5 OUTB, J6 CAN-HI, J7 CAN-LO, P1 Digital, P2 Analog, P3 CONN_01X01, P4 CONN_01X01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

Commit message: many changes
Parts:
- added D1: PMEG3020EH, Diodes_SMD:D_SOD-123F, symbol Diode:PMEG3020EH
- added F1: 15A, CustomComponents:atm_fuse_holder-mpd-bk-6013, symbol Device:Fuse
- added H6, H7, H8, H9: MountingHole, Mounting_Holes:MountingHole_3.2mm_M3, symbol Mechanical:MountingHole
- added J1: Right Rudder Stop, Connectors_JST:JST_XH_B02B-XH-A_02x2.50mm_Straight, symbol Connector_Generic:Conn_01x02
- added J8: Left Rudder Stop, Connectors_JST:JST_XH_B02B-XH-A_02x2.50mm_Straight, symbol Connector_Generic:Conn_01x02
Connections:
- net +12V: now also D1.2 (A), F1.2; no longer J2.1 (Pin_1)
- net D7: now also J1.1 (Pin_1)
- net D8: now also J8.1 (Pin_1)
- net GND: now also J1.2 (Pin_2), J8.2 (Pin_2)
- net Vin: now also D1.1 (K)
- net 0(Rx) renamed Rx
- net 1(Tx) renamed Tx
- new net: F1.1, J2.1 (Pin_1)
- no-connect marks 11 -> 12
Other:
- note added: "CAN Bus"
- note added: "Faston Connectors"
- note added: "Motor Controller"
- note added: "Mounting Holes"
- note added: "Rudder Stop Switches"
Changed lines of the file:
@@
 $EndDescr
 Text Label 8025 1075 0    60   ~ 0
-1(Tx)
+Tx
 Text Label 8025 1175 0    60   ~ 0
-0(Rx)
+Rx
 Text Label 8025 1275 0    60   ~ 0
 Reset
@@
 Wire Wire Line
 	6850 4375 6550 4375
-Text GLabel 6550 4475 0    50   Input ~ 0
+Text GLabel 6550 4475 0    50   Output ~ 0
 A1
 Wire Wire Line
@@
 Text GLabel 6550 4175 0    50   Input ~ 0
 D2
-Text GLabel 6550 4275 0    50   Input ~ 0
+Text GLabel 6550 4275 0    50   BiDi ~ 0
 D4
 Wire Wire Line
@@
 Wire Wire Line
 	6550 4675 6850 4675
-Text GLabel 6550 4575 0    50   Input ~ 0
+Text GLabel 6550 4575 0    50   BiDi ~ 0
 D5
 Wire Wire Line
@@
 L power:+12V #PWR0116
 U 1 1 607384B9
-P 5800 1275
-F 0 "#PWR0116" H 5800 1125 50  0001 C CNN
-F 1 "+12V" H 5815 1448 50  0000 C CNN
-F 2 "" H 5800 1275 50  0001 C CNN
-F 3 "" H 5800 1275 50  0001 C CNN
-	1    5800 1275
+P 5550 975
+F 0 "#PWR0116" H 5550 825 50  0001 C CNN
+F 1 "+12V" H 5565 1148 50  0000 C CNN
+F 2 "" H 5550 975 50  0001 C CNN
+F 3 "" H 5550 975 50  0001 C CNN
+	1    5550 975
 	1    0    0    -1
 $EndComp
@@
 Wire Wire Line
 	5800 1625 5900 1625
-Wire Wire Line
-	5800 1275 5900 1275
 $Comp
 L Connector_Generic:Conn_01x01 J2
@@
 Wire Wire Line
 	5800 2800 5900 2800
+$Comp
+L Mechanical:MountingHole H6
+U 1 1 6076CA7C
+P 2475 1575
+F 0 "H6" H 2575 1621 50  0000 L CNN
+F 1 "MountingHole" H 2575 1530 50  0000 L CNN
+F 2 "Mounting_Holes:MountingHole_3.2mm_M3" H 2475 1575 50  0001 C CNN
+F 3 "~" H 2475 1575 50  0001 C CNN
+	1    2475 1575
+	1    0    0    -1
+$EndComp
+$Comp
+L Mechanical:MountingHole H7
+U 1 1 6076DA94
+P 3275 1550
+F 0 "H7" H 3375 1596 50  0000 L CNN
+F 1 "MountingHole" H 3375 1505 50  0000 L CNN
+F 2 "Mounting_Holes:MountingHole_3.2mm_M3" H 3275 1550 50  0001 C CNN
+F 3 "~" H 3275 1550 50  0001 C CNN
+	1    3275 1550
+	1    0    0    -1
+$EndComp
+$Comp
+L Mechanical:MountingHole H8
+U 1 1 6076DD76
+P 2475 1825
+F 0 "H8" H 2575 1871 50  0000 L CNN
+F 1 "MountingHole" H 2575 1780 50  0000 L CNN
+F 2 "Mounting_Holes:MountingHole_3.2mm_M3" H 2475 1825 50  0001 C CNN
+F 3 "~" H 2475 1825 50  0001 C CNN
+	1    2475 1825
+	1    0    0    -1
+$EndComp
+$Comp
+L Mechanical:MountingHole H9
+U 1 1 6076E12C
+P 3275 1800
+F 0 "H9" H 3375 1846 50  0000 L CNN
+F 1 "MountingHole" H 3375 1755 50  0000 L CNN
+F 2 "Mounting_Holes:MountingHole_3.2mm_M3" H 3275 1800 50  0001 C CNN
+F 3 "~" H 3275 1800 50  0001 C CNN
+	1    3275 1800
+	1    0    0    -1
+$EndComp
+$Comp
+L Diode:PMEG3020EH D1
+U 1 1 6079E0C1
+P 5225 1275
+F 0 "D1" H 5225 1491 50  0000 C CNN
+F 1 "PMEG3020EH" H 5225 1400 50  0000 C CNN
+F 2 "Diodes_SMD:D_SOD-123F" H 5225 1100 50  0001 C CNN
+F 3 "https://assets.nexperia.com/documents/data-sheet/PMEG3020EH_EJ.pdf" H 5225 1275 50  0001 C CNN
+	1    5225 1275
+	1    0    0    -1
+$EndComp
+Wire Wire Line
+	5075 1275 4575 1275
+Text Label 4575 1275 0    50   ~ 0
+Vin
+NoConn ~ 6850 4875
+$Comp
+L Device:Fuse F1
+U 1 1 6080C892
+P 5700 1275
+F 0 "F1" V 5503 1275 50  0000 C CNN
+F 1 "15A" V 5594 1275 50  0000 C CNN
+F 2 "CustomComponents:atm_fuse_holder-mpd-bk-6013" V 5630 1275 50  0001 C CNN
+F 3 "~" H 5700 1275 50  0001 C CNN
+	1    5700 1275
+	0    1    1    0
+$EndComp
+Wire Wire Line
+	5375 1275 5550 1275
+Wire Wire Line
+	5550 1275 5550 975
+Connection ~ 5550 1275
+Wire Wire Line
+	5850 1275 5900 1275
+Text Notes 2725 1375 0    50   ~ 10
+Mounting Holes
+Text Notes 3100 3050 0    50   ~ 10
+CAN Bus
+Text Notes 7575 3650 0    50   ~ 10
+Motor Controller
+Text Notes 5750 950  0    50   ~ 10
+Faston Connectors
+$Comp
+L Connector_Generic:Conn_01x02 J1
+U 1 1 60871480
+P 2675 6050
+F 0 "J1" H 2755 6042 50  0000 L CNN
+F 1 "Right Rudder Stop" H 2755 5951 50  0000 L CNN
+F 2 "Connectors_JST:JST_XH_B02B-XH-A_02x2.50mm_Straight" H 2675 6050 50  0001 C CNN
+F 3 "~" H 2675 6050 50  0001 C CNN
+	1    2675 6050
+	1    0    0    -1
+$EndComp
+$Comp
+L Connector_Generic:Conn_01x02 J8
+U 1 1 6087706D
+P 2675 6425
+F 0 "J8" H 2755 6417 50  0000 L CNN
+F 1 "Left Rudder Stop" H 2755 6326 50  0000 L CNN
+F 2 "Connectors_JST:JST_XH_B02B-XH-A_02x2.50mm_Straight" H 2675 6425 50  0001 C CNN
+F 3 "~" H 2675 6425 50  0001 C CNN
+	1    2675 6425
+	1    0    0    -1
+$EndComp
+$Comp
+L power:GND #PWR?
+U 1 1 6087F73E
+P 2125 6525
+F 0 "#PWR?" H 2125 6275 50  0001 C CNN
+F 1 "GND" H 2130 6352 50  0000 C CNN
+F 2 "" H 2125 6525 50  0001 C CNN
+F 3 "" H 2125 6525 50  0001 C CNN
+	1    2125 6525
+	1    0    0    -1
+$EndComp
+Wire Wire Line
+	2475 6525 2125 6525
+Wire Wire Line
+	2475 6150 2125 6150
+Wire Wire Line
+	2125 6150 2125 6525
+Connection ~ 2125 6525
+Text GLabel 2375 6050 0    50   Input ~ 0
+D7
+Text GLabel 2375 6425 0    50   Input ~ 0
+D8
+Wire Wire Line
+	2375 6050 2475 6050
+Wire Wire Line
+	2375 6425 2475 6425
+Text Notes 2400 5875 0    50   ~ 10
+Rudder Stop Switches
 $EndSCHEMATC

Commit message: Crystal was wired incorrectly
Replaced schematic symbol
Fixed pcb layout
incremented revision to B
Parts:
- removed Y1: 16MHz, Crystals:Crystal_SMD_TXC_7M-4pin_3.2x2.5mm, symbol Device:Crystal
- added Y1: 16MHz, Crystals:Crystal_SMD_TXC_7M-4pin_3.2x2.5mm, symbol Device:Crystal_GND24
Connections:
- net GND: now also Y1.2, Y1.4
- net at C3.1, U1.7 (OSC2): now also Y1.1
- net at C4.1, U1.8 (OSC1): now also Y1.3
Changed lines of the file:
@@
 Title "PyPilot Controller"
 Date "2021 April 10"
-Rev "A"
+Rev "B"
 Comp "bit-builder.com"
 Comment1 ""
@@
 $EndComp
 $Comp
-L Device:Crystal Y1
-U 1 1 60730883
-P 1075 4400
-F 0 "Y1" H 1075 4668 50  0000 C CNN
-F 1 "16MHz" H 1075 4577 50  0000 C CNN
-F 2 "Crystals:Crystal_SMD_TXC_7M-4pin_3.2x2.5mm" H 1075 4400 50  0001 C CNN
-F 3 "~" H 1075 4400 50  0001 C CNN
-	1    1075 4400
-	1    0    0    -1
-$EndComp
-$Comp
 L power:+12V #PWR0102
 U 1 1 6073212C
@@
 $EndComp
 Wire Wire Line
-	1600 4200 925  4200
-Wire Wire Line
-	925  4200 925  4400
-Wire Wire Line
 	1600 4300 1225 4300
 Wire Wire Line
@@
 Wire Wire Line
 	800  4400 800  4625
-Connection ~ 925  4400
 Wire Wire Line
 	1225 4400 1325 4400
 Wire Wire Line
 	1325 4400 1325 4625
-Connection ~ 1225 4400
 Wire Wire Line
 	2200 4800 2200 4875
@@
 Text Notes 2400 5875 0    50   ~ 10
 Rudder Stop Switches
+$Comp
+L Device:Crystal_GND24 Y1
+U 1 1 6083F2DE
+P 1075 4400
+F 0 "Y1" H 1269 4446 50  0000 L CNN
+F 1 "16MHz" H 1269 4355 50  0000 L CNN
+F 2 "Crystals:Crystal_SMD_TXC_7M-4pin_3.2x2.5mm" H 1075 4400 50  0001 C CNN
+F 3 "~" H 1075 4400 50  0001 C CNN
+	1    1075 4400
+	1    0    0    -1
+$EndComp
+Connection ~ 1225 4400
+Wire Wire Line
+	800  4400 800  4075
+Wire Wire Line
+	800  4075 1350 4075
+Wire Wire Line
+	1350 4075 1350 4200
+Wire Wire Line
+	1350 4200 1600 4200
+Connection ~ 800  4400
+$Comp
+L power:GND #PWR?
+U 1 1 6084D80E
+P 650 4200
+F 0 "#PWR?" H 650 3950 50  0001 C CNN
+F 1 "GND" H 655 4027 50  0000 C CNN
+F 2 "" H 650 4200 50  0001 C CNN
+F 3 "" H 650 4200 50  0001 C CNN
+	1    650  4200
+	1    0    0    -1
+$EndComp
+Wire Wire Line
+	1075 4600 1075 5025
+Wire Wire Line
+	1075 4200 650  4200
 $EndSCHEMATC
